Commit message: Should have corrected the warning/issue with gazebo.

File: dabom_ws/src/dabomb_description/urdf/dabomb.xacro (robot description, xacro)
@@ -155,5 +155,5 @@
 </joint>
 <joint name="laser_joint" type="fixed">
-  <origin xyz="0.0 0.0 0.15" rpy="0 0 0"/>
+  <origin xyz="0.0 0.0 0.15" rpy="0 0 3.1415926"/>
   <parent link="base_link"/>
   <child link="laser"/>

Commit message: rotated laser forwards

File: dabom_ws/src/dabomb_description/urdf/dabomb.xacro (robot description, xacro)
@@ -155,5 +155,5 @@
 </joint>
 <joint name="laser_joint" type="fixed">
-  <origin xyz="0.0 0.0 0.15" rpy="0 0 3.1415926"/>
+  <origin xyz="0.0 0.0 0.15" rpy="0 0 0"/>
   <parent link="base_link"/>
   <child link="laser"/>

Commit message: aaded euler to quaternion

File: dabom_ws/src/dabomb_description/urdf/dabomb.xacro (robot description, xacro)
@@ -155,5 +155,5 @@
 </joint>
 <joint name="laser_joint" type="fixed">
-  <origin xyz="0.0 0.0 0.15" rpy="0 0 0"/>
+  <origin xyz="0.0 0.0 0.15" rpy="0 0 3.14159"/>
   <parent link="base_link"/>
   <child link="laser"/>

Commit message: rotated laser back to 0

File: dabom_ws/src/dabomb_description/urdf/dabomb.xacro (robot description, xacro)
@@ -155,5 +155,5 @@
 </joint>
 <joint name="laser_joint" type="fixed">
-  <origin xyz="0.0 0.0 0.15" rpy="0 0 3.14159"/>
+  <origin xyz="0.0 0.0 0.15" rpy="0 0 0"/>
   <parent link="base_link"/>
   <child link="laser"/>

Commit message: rotated 180

File: dabom_ws/src/dabomb_description/urdf/dabomb.xacro (robot description, xacro)
@@ -155,5 +155,5 @@
 </joint>
 <joint name="laser_joint" type="fixed">
-  <origin xyz="0.0 0.0 0.15" rpy="0 0 0"/>
+  <origin xyz="0.0 0.0 0.15" rpy="0 0 3.14"/>
   <parent link="base_link"/>
   <child link="laser"/>

Commit message: rotated laser to 0 degrees

File: dabom_ws/src/dabomb_description/urdf/dabomb.xacro (robot description, xacro)
@@ -155,5 +155,5 @@
 </joint>
 <joint name="laser_joint" type="fixed">
-  <origin xyz="0.0 0.0 0.15" rpy="0 0 3.14"/>
+  <origin xyz="0.0 0.0 0.15" rpy="0 0 0"/>
   <parent link="base_link"/>
   <child link="laser"/>

Commit message: Changed URDF laser from 3.14 to pi

File: dabom_ws/src/dabomb_description/urdf/dabomb.xacro (robot description, xacro)
@@ -158,5 +158,5 @@
 </joint>
 <joint name="laser_joint" type="fixed">
-  <origin xyz="0.0 0.0 0.15" rpy="0 0 3.14"/>
+  <origin xyz="0.0 0.0 0.15" rpy="0 0 ${pi}"/>
   <parent link="base_link"/>
   <child link="laser"/>

Commit message: gazebo working

File: dabom_ws/src/dabomb_description/urdf/dabomb.xacro (robot description, xacro)
@@ -138,4 +138,7 @@
   <child link="Wheel1_1"/>
   <axis xyz="-0.0 1.0 0.0"/>
+  <joint_properties damping="100" friction="1000"/>
+  <limit effort="1000.0" lower="-1e+16" upper="1e+16" velocity="10"/>
+  <joint_properties damping="1.0" friction="1"/>
 </joint>
 <joint name="Wheel3" type="continuous">
@@ -144,4 +147,7 @@
   <child link="Wheel3_1"/>
   <axis xyz="0.0 1.0 0.0"/>
+  <joint_properties damping="100" friction="1000"/>
+  <limit effort="1000.0" lower="-1e+16" upper="1e+16" velocity="10"/>
+  <joint_properties damping="1.0" friction="1"/>
 </joint>
 <joint name="Wheel2" type="continuous">
@@ -150,4 +156,7 @@
   <child link="Wheel2_1"/>
   <axis xyz="-0.0 -1.0 0.0"/>
+  <joint_properties damping="100" friction="1000"/>
+  <limit effort="1000.0" lower="-1e+16" upper="1e+16" velocity="10"/>
+  <joint_properties damping="1.0" friction="1"/>
 </joint>
 <joint name="Wheel4" type="continuous">
@@ -156,4 +165,7 @@
   <child link="Wheel4_1"/>
   <axis xyz="0.0 -1.0 0.0"/>
+  <joint_properties damping="100" friction="1000"/>
+  <limit effort="1000.0" lower="-1e+16" upper="1e+16" velocity="10"/>
+  <joint_properties damping="1.0" friction="1"/>
 </joint>
 <joint name="laser_joint" type="fixed">
@@ -161,4 +173,7 @@
   <parent link="base_link"/>
   <child link="laser"/>
+  <joint_properties damping="100" friction="1000"/>
+  <limit effort="1000.0" lower="-1e+16" upper="1e+16" velocity="10"/>
+  <joint_properties damping="1.0" friction="1"/>
 </joint>
 </robot>
